File: projects/CanSat/Czopolot 1.0/schematic.brd (EAGLE design)
At the start: 115 x 66 mm, 6 parts

Commit message: File update
Parts:
- U$1: device PyBoard 1.1 footprint:PYBOARD -> SobieskiSat2:MODULE_PYBOARD
Changed lines of the file:
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@@
 </autorouter>
 <elements>
-<element name="U$1" library="PyBoard 1.1 footprint" package="PYBOARD" value="PYBOARD1.1" x="-10.16" y="-8.89" smashed="yes"/>
+<element name="U$1" library="SobieskiSat2" package="MODULE_PYBOARD" value="PYBOARD1.1" x="-10.16" y="-8.89" smashed="yes"/>
 <element name="ULTIMATE_GPS" library="pinhead" library_urn="urn:adsk.eagle:library:325" package="1X04" package3d_urn="urn:adsk.eagle:package:22407/2" value="" x="-19.05" y="-5.08" smashed="yes" rot="R90">
 <attribute name="NAME" x="-20.8788" y="-10.2362" size="1.27" layer="25" ratio="10" rot="R90"/>

Commit message: Work work..
Parts:
- U$2: value SX1280EXT -> SX1280; device SobieskiSat2:MODULE_SX1280_EXT -> SobieskiSat2:MODULE_SX1280
Connections:
- new net BAT+: U$1.VBAT
- new net DIO1: U$1.X3, U$2.DIO1
Changed lines of the file:
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@@
 <attribute name="VALUE" x="-15.875" y="-10.16" size="1.27" layer="27" rot="R90"/>
 </element>
-<element name="U$2" library="SobieskiSat2" package="MODULE_SX1280_EXT" value="SX1280EXT" x="1.27" y="-16.51" smashed="yes" rot="R270"/>
+<element name="U$2" library="SobieskiSat2" package="MODULE_SX1280" value="SX1280" x="1.27" y="-16.51" smashed="yes" rot="R270"/>
 <element name="X1" library="SobieskiSat2" package="SMA_DIP" package3d_urn="urn:adsk.eagle:package:6240946/1" value="" x="-11.43" y="-19.05" smashed="yes">
 <attribute name="NAME" x="-13.462" y="-14.224" size="0.8128" layer="25" ratio="18"/>
@@
 <wire x1="-16.51" y1="-3.81" x2="-19.05" y2="-3.81" width="0" layer="19" extent="1-1"/>
 </signal>
-<signal name="GND" airwireshidden="yes">
+<signal name="GND">
 <contactref element="ULTIMATE_GPS" pad="2"/>
 <contactref element="U$2" pad="GND@1"/>
@@
 <wire x1="-6.35" y1="-34.289" x2="-16.51" y2="-24.13" width="0" layer="19" extent="1-1"/>
 </signal>
+<signal name="BAT+">
+<contactref element="U$1" pad="VBAT"/>
+</signal>
+<signal name="BAT-">
+</signal>
+<signal name="DIO1">
+<contactref element="U$2" pad="DIO1"/>
+<contactref element="U$1" pad="X3"/>
+<wire x1="8.27" y1="-23.51" x2="11.43" y2="-34.29" width="0" layer="19" extent="1-1"/>
+</signal>
 </signals>
