File: projects/CanSat/Czopolot 1.0/schematic.brd (EAGLE design)
At the start: 115 x 66 mm, 6 parts

Commit message: Work work..
Parts:
- added JP1, JP2: (no value), pinhead:1X02
- added Q1, Q2: (no value), adafruit:TO220V
- added R1, R2: (no value), rcl:0207/10
Changed lines of the file:
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@@
 <element name="U$3" library="SobieskiSat2" package="MODULE_MPU9250" value="MPU9250" x="-2.54" y="-8.001" smashed="yes" rot="R270"/>
 <element name="U$4" library="SobieskiSat2" package="MODULE_BMP280" value="BMP280" x="-7.62" y="-28.829" smashed="yes" rot="R90"/>
+<element name="R1" library="rcl" library_urn="urn:adsk.eagle:library:334" package="0207/10" package3d_urn="urn:adsk.eagle:package:23491/2" value="" x="-62.23" y="-52.07" smashed="yes" rot="R90">
+<attribute name="NAME" x="-63.754" y="-55.118" size="1.27" layer="25" ratio="10" rot="R90"/>
+<attribute name="POPULARITY" value="81" x="-62.23" y="-52.07" size="1.778" layer="27" rot="R90" display="off"/>
+<attribute name="SPICEPREFIX" value="R" x="-62.23" y="-52.07" size="1.778" layer="27" rot="R90" display="off"/>
+<attribute name="VALUE" x="-61.595" y="-54.3306" size="1.27" layer="27" ratio="10" rot="R90"/>
+</element>
+<element name="R2" library="rcl" library_urn="urn:adsk.eagle:library:334" package="0207/10" package3d_urn="urn:adsk.eagle:package:23491/2" value="" x="-67.31" y="-52.07" smashed="yes" rot="R90">
+<attribute name="NAME" x="-68.834" y="-55.118" size="1.27" layer="25" ratio="10" rot="R90"/>
+<attribute name="POPULARITY" value="81" x="-67.31" y="-52.07" size="1.778" layer="27" rot="R90" display="off"/>
+<attribute name="SPICEPREFIX" value="R" x="-67.31" y="-52.07" size="1.778" layer="27" rot="R90" display="off"/>
+<attribute name="VALUE" x="-66.675" y="-54.3306" size="1.27" layer="27" ratio="10" rot="R90"/>
+</element>
+<element name="Q1" library="adafruit" library_urn="urn:adsk.eagle:library:420" package="TO220V" package3d_urn="urn:adsk.eagle:package:6240882/1" value="" x="-63.5" y="-35.56" smashed="yes" rot="R90">
+<attribute name="NAME" x="-57.4548" y="-40.64" size="1.27" layer="25" ratio="10" rot="R90"/>
+<attribute name="VALUE" x="-55.88" y="-40.64" size="1.27" layer="27" ratio="10" rot="R90"/>
+</element>
+<element name="Q2" library="adafruit" library_urn="urn:adsk.eagle:library:420" package="TO220V" package3d_urn="urn:adsk.eagle:package:6240882/1" value="" x="-63.5" y="-20.32" smashed="yes" rot="R90">
+<attribute name="NAME" x="-57.4548" y="-25.4" size="1.27" layer="25" ratio="10" rot="R90"/>
+<attribute name="VALUE" x="-55.88" y="-25.4" size="1.27" layer="27" ratio="10" rot="R90"/>
+</element>
+<element name="JP1" library="pinhead" library_urn="urn:adsk.eagle:library:325" package="1X02" package3d_urn="urn:adsk.eagle:package:22435/2" value="" x="-53.34" y="-60.96" smashed="yes">
+<attribute name="NAME" x="-55.9562" y="-59.1312" size="1.27" layer="25" ratio="10"/>
+<attribute name="POPULARITY" value="98" x="-53.34" y="-60.96" size="1.778" layer="27" display="off"/>
+<attribute name="VALUE" x="-55.88" y="-64.135" size="1.27" layer="27"/>
+</element>
+<element name="JP2" library="pinhead" library_urn="urn:adsk.eagle:library:325" package="1X02" package3d_urn="urn:adsk.eagle:package:22435/2" value="" x="-43.18" y="-60.96" smashed="yes">
+<attribute name="NAME" x="-45.7962" y="-59.1312" size="1.27" layer="25" ratio="10"/>
+<attribute name="POPULARITY" value="98" x="-43.18" y="-60.96" size="1.778" layer="27" display="off"/>
+<attribute name="VALUE" x="-45.72" y="-64.135" size="1.27" layer="27"/>
+</element>
 </elements>
 <signals>

Commit message: Work work..
Parts:
- moved JP1 37.8 mm to (-17.8, -48.3)
- moved JP2 37.8 mm to (-7.62, -48.3)
- moved Q1 37.8 mm to (-27.9, -22.9)
- moved Q2 37.8 mm to (-27.9, -7.62)
- moved R2 37.8 mm to (-31.8, -39.4)
- moved R1 37.8 mm to (-26.7, -39.4)
- moved U$2 25.5 mm to (26.7, -19.1)
- moved U$4 25.5 mm to (17.8, -31.4)
- moved U$1 25.5 mm to (15.2, -11.4)
- moved U$3 25.5 mm to (22.9, -10.5)
- moved ULTIMATE_GPS 25.5 mm to (6.35, -7.62)
- moved X1 25.5 mm to (14.0, -21.6)
Other:
- board size 115 x 66 mm -> 43.2 x 48.3 mm

Commit message: Work work..
Parts:
- moved Q1 9.16 mm to (-20.3, -27.9)
- moved JP1 2.54 mm to (-17.8, -45.7)
Connections:
- new net V+: U$1.V+, U$1.V+1, U$1.V+2, U$1.V+3, U$1.V+4, U$1.V+5, U$1.V+6, ULTIMATE_GPS.1
- net VCC: no longer ULTIMATE_GPS.1
Changed lines of the file:
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@@
 <attribute name="VALUE" x="-31.115" y="-41.6306" size="1.27" layer="27" ratio="10" rot="R90"/>
 </element>
-<element name="Q1" library="adafruit" library_urn="urn:adsk.eagle:library:420" package="TO220V" package3d_urn="urn:adsk.eagle:package:6240882/1" value="" x="-27.94" y="-22.86" smashed="yes" rot="R90">
-<attribute name="NAME" x="-21.8948" y="-27.94" size="1.27" layer="25" ratio="10" rot="R90"/>
-<attribute name="VALUE" x="-20.32" y="-27.94" size="1.27" layer="27" ratio="10" rot="R90"/>
+<element name="Q1" library="adafruit" library_urn="urn:adsk.eagle:library:420" package="TO220V" package3d_urn="urn:adsk.eagle:package:6240882/1" value="" x="-20.32" y="-27.94" smashed="yes" rot="R90">
+<attribute name="NAME" x="-14.2748" y="-33.02" size="1.27" layer="25" ratio="10" rot="R90"/>
+<attribute name="VALUE" x="-12.7" y="-33.02" size="1.27" layer="27" ratio="10" rot="R90"/>
 </element>
 <element name="Q2" library="adafruit" library_urn="urn:adsk.eagle:library:420" package="TO220V" package3d_urn="urn:adsk.eagle:package:6240882/1" value="" x="-27.94" y="-7.62" smashed="yes" rot="R90">
@@
 <attribute name="VALUE" x="-20.32" y="-12.7" size="1.27" layer="27" ratio="10" rot="R90"/>
 </element>
-<element name="JP1" library="pinhead" library_urn="urn:adsk.eagle:library:325" package="1X02" package3d_urn="urn:adsk.eagle:package:22435/2" value="" x="-17.78" y="-48.26" smashed="yes">
-<attribute name="NAME" x="-20.3962" y="-46.4312" size="1.27" layer="25" ratio="10"/>
-<attribute name="POPULARITY" value="98" x="-17.78" y="-48.26" size="1.778" layer="27" display="off"/>
-<attribute name="VALUE" x="-20.32" y="-51.435" size="1.27" layer="27"/>
+<element name="JP1" library="pinhead" library_urn="urn:adsk.eagle:library:325" package="1X02" package3d_urn="urn:adsk.eagle:package:22435/2" value="" x="-17.78" y="-45.72" smashed="yes">
+<attribute name="NAME" x="-20.3962" y="-43.8912" size="1.27" layer="25" ratio="10"/>
+<attribute name="POPULARITY" value="98" x="-17.78" y="-45.72" size="1.778" layer="27" display="off"/>
+<attribute name="VALUE" x="-20.32" y="-48.895" size="1.27" layer="27"/>
 </element>
 <element name="JP2" library="pinhead" library_urn="urn:adsk.eagle:library:325" package="1X02" package3d_urn="urn:adsk.eagle:package:22435/2" value="" x="-7.62" y="-48.26" smashed="yes">
@@
 <contactref element="U$3" pad="VCC"/>
 <contactref element="U$4" pad="VCC"/>
-<contactref element="ULTIMATE_GPS" pad="1"/>
 <contactref element="U$1" pad="3V3-1"/>
 <contactref element="U$1" pad="3V3"/>
 <wire x1="36.83" y1="-6.35" x2="34.29" y2="-3.811" width="0" layer="19" extent="1-1"/>
 <wire x1="29.67" y1="-12.05" x2="36.83" y2="-6.35" width="0" layer="19" extent="1-1"/>
-<wire x1="6.35" y1="-11.43" x2="29.67" y2="-12.05" width="0" layer="19" extent="1-1"/>
-<wire x1="11.43" y1="-36.829" x2="6.35" y2="-11.43" width="0" layer="19" extent="1-1"/>
+<wire x1="11.43" y1="-36.829" x2="29.67" y2="-12.05" width="0" layer="19" extent="1-1"/>
 <wire x1="8.89" y1="-39.37" x2="11.43" y2="-36.829" width="0" layer="19" extent="1-1"/>
 </signal>
@@
 <wire x1="36.83" y1="-36.83" x2="33.67" y2="-26.05" width="0" layer="19" extent="1-1"/>
 </signal>
+<signal name="V+">
+<contactref element="U$1" pad="V+3"/>
+<contactref element="U$1" pad="V+2"/>
+<contactref element="U$1" pad="V+"/>
+<contactref element="U$1" pad="V+4"/>
+<contactref element="U$1" pad="V+5"/>
+<contactref element="U$1" pad="V+6"/>
+<contactref element="U$1" pad="V+1"/>
+<contactref element="ULTIMATE_GPS" pad="1"/>
+<wire x1="34.29" y1="-34.29" x2="36.83" y2="-3.81" width="0" layer="19" extent="1-1"/>
+<wire x1="34.29" y1="-36.83" x2="34.29" y2="-34.29" width="0" layer="19" extent="1-1"/>
+<wire x1="34.29" y1="-39.37" x2="34.29" y2="-36.83" width="0" layer="19" extent="1-1"/>
+<wire x1="34.29" y1="-41.91" x2="34.29" y2="-39.37" width="0" layer="19" extent="1-1"/>
+<wire x1="26.67" y1="-39.37" x2="34.29" y2="-39.37" width="0" layer="19" extent="1-1"/>
+<wire x1="8.89" y1="-41.91" x2="26.67" y2="-39.37" width="0" layer="19" extent="1-1"/>
+<wire x1="6.35" y1="-11.43" x2="8.89" y2="-41.91" width="0" layer="19" extent="1-1"/>
+</signal>
 </signals>

Commit message: Work work..
Parts:
- moved Q2 55.8 mm to (8.89, -49.5), turned to 180 degrees
- moved R1 53.4 mm to (26.7, -41.9), turned to 180 degrees
- moved Q1 51.7 mm to (26.7, -49.5), turned to 180 degrees
- moved JP2 41.9 mm to (34.3, -48.3), turned to 90 degrees
- moved R2 40.7 mm to (8.89, -41.9), turned to 180 degrees
- moved JP1 19.2 mm to (1.27, -48.3), turned to 90 degrees
- moved U$2 3.59 mm to (24.1, -16.5)
- moved U$1 3.59 mm to (12.7, -8.89)
- moved U$3 3.59 mm to (20.3, -8.00)
- moved U$4 3.59 mm to (15.2, -28.8)
- moved ULTIMATE_GPS 3.59 mm to (3.81, -5.08)
- moved X1 3.59 mm to (11.4, -19.1)
Other:
- board size 43.2 x 48.3 mm -> 35.6 x 50.8 mm
