File: projects/CanSat/ExpansionBoard/ExpansionBoard.sch (EAGLE design)
At the start: 32 parts, among them X1 FH12-24S-0.5SH

Commit message: Before ordering
Connections:
- net GND: now also X1-18.1, X1-24.1; no longer X1-17.1, X1-23.1
- net VCC: now also X1-17.1, X1-23.1; no longer X1-18.1, X1-24.1
Changed lines of the file:
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@@
 <setting verticaltext="up"/>
 </settings>
-<grid distance="0.1" unitdist="inch" unit="inch" style="lines" multiple="1" display="no" altdistance="0.01" altunitdist="inch" altunit="inch"/>
+<grid distance="0.05" unitdist="inch" unit="inch" style="lines" multiple="1" display="no" altdistance="0.01" altunitdist="inch" altunit="inch"/>
 <layers>
 <layer number="1" name="Top" color="4" fill="1" visible="no" active="no"/>
@@
 <instance part="U$21" gate="G$1" x="15.24" y="-20.32" smashed="yes" rot="R180"/>
 <instance part="U$22" gate="G$1" x="15.24" y="-22.86" smashed="yes" rot="R180"/>
-<instance part="U$23" gate="G$1" x="15.24" y="-25.4" smashed="yes" rot="R180"/>
-<instance part="U$24" gate="G$1" x="15.24" y="-27.94" smashed="yes" rot="R180"/>
+<instance part="U$23" gate="G$1" x="15.24" y="-27.94" smashed="yes" rot="R180"/>
+<instance part="U$24" gate="G$1" x="15.24" y="-25.4" smashed="yes" rot="R180"/>
 <instance part="X1" gate="G$2" x="38.1" y="-33.02" smashed="yes"/>
 <instance part="U$28" gate="G$1" x="-20.32" y="5.08" smashed="yes"/>
@@
 </segment>
 <segment>
-<pinref part="X1" gate="-17" pin="1"/>
-<wire x1="19.05" y1="-10.16" x2="35.56" y2="-10.16" width="0.1524" layer="91"/>
-<label x="20.32" y="-10.16" size="1.778" layer="95"/>
-</segment>
-<segment>
-<pinref part="X1" gate="-23" pin="1"/>
-<pinref part="U$23" gate="G$1" pin="1"/>
-<wire x1="19.05" y1="-25.4" x2="35.56" y2="-25.4" width="0.1524" layer="91"/>
-<label x="20.32" y="-25.4" size="1.778" layer="95"/>
-</segment>
-<segment>
 <wire x1="-17.78" y1="22.86" x2="-19.05" y2="22.86" width="0.1524" layer="91"/>
 <label x="-19.05" y="22.86" size="0.762" layer="95" rot="R180" xref="yes"/>
@@
 <label x="30.48" y="-33.02" size="0.762" layer="95" rot="R180" xref="yes"/>
 </segment>
+<segment>
+<wire x1="19.05" y1="-12.7" x2="35.56" y2="-12.7" width="0.1524" layer="91"/>
+<label x="20.32" y="-12.7" size="1.778" layer="95"/>
+<pinref part="X1" gate="-18" pin="1"/>
+</segment>
+<segment>
+<pinref part="X1" gate="-24" pin="1"/>
+<pinref part="U$23" gate="G$1" pin="1"/>
+<wire x1="19.05" y1="-27.94" x2="35.56" y2="-27.94" width="0.1524" layer="91"/>
+<label x="20.32" y="-27.94" size="1.778" layer="95"/>
+</segment>
 </net>
 <net name="VCC" class="0">
@@
 <wire x1="19.05" y1="12.7" x2="35.56" y2="12.7" width="0.1524" layer="91"/>
 <label x="20.32" y="12.7" size="1.778" layer="95"/>
-</segment>
-<segment>
-<pinref part="X1" gate="-18" pin="1"/>
-<wire x1="19.05" y1="-12.7" x2="35.56" y2="-12.7" width="0.1524" layer="91"/>
-<label x="20.32" y="-12.7" size="1.778" layer="95"/>
-</segment>
-<segment>
-<pinref part="X1" gate="-24" pin="1"/>
-<pinref part="U$24" gate="G$1" pin="1"/>
-<wire x1="19.05" y1="-27.94" x2="35.56" y2="-27.94" width="0.1524" layer="91"/>
-<label x="20.32" y="-27.94" size="1.778" layer="95"/>
 </segment>
 <segment>
@@
 <label x="-71.12" y="-15.24" size="0.762" layer="95" xref="yes"/>
 </segment>
+<segment>
+<wire x1="19.05" y1="-10.16" x2="35.56" y2="-10.16" width="0.1524" layer="91"/>
+<label x="20.32" y="-10.16" size="1.778" layer="95"/>
+<pinref part="X1" gate="-17" pin="1"/>
+</segment>
+<segment>
+<pinref part="X1" gate="-23" pin="1"/>
+<pinref part="U$24" gate="G$1" pin="1"/>
+<wire x1="19.05" y1="-25.4" x2="35.56" y2="-25.4" width="0.1524" layer="91"/>
+<label x="20.32" y="-25.4" size="1.778" layer="95"/>
+</segment>
 </net>
