File: projects/CanSat/ExpansionBoard/ExpansionBoard.brd (EAGLE design)
At the start: 17.8 x 33.7 mm, 32 parts, among them X1 FH12-24S-0.5SH

Commit message: Before ordering
Parts:
- moved C1 0.60 mm to (4.09, 23.2)
- moved C2 0.60 mm to (13.7, 23.2)
Connections:
- net GND: now also X1.18, X1.24; no longer X1.17, X1.23
- net VCC: now also X1.17, X1.23; no longer X1.18, X1.24
Routing:
- net VCC: track 58.2 -> 65.8 mm
- net GND: track 45.0 -> 39.0 mm, vias 18 -> 17
