File: projects/CanSat/Czopolot 2.0/Schematic.sch (EAGLE design)
At the start: 95 parts, among them X1 FH12-24S-0.5SH

Commit message: GND yet to fix
Connections:
- net BAT: now also C28.+, U$19.S$1
- net GND: now also C28.-; no longer U$19.S$1
Changed lines of the file:
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@@
 <part name="P+7" library="supply1" library_urn="urn:adsk.eagle:library:371" deviceset="VCC" device=""/>
 <part name="C80" library="Unified" deviceset="CAPACITOR" device="0603" package3d_urn="urn:adsk.eagle:package:23616/2" value="10u"/>
-<part name="BTN_RST" library="SobieskiSat2" deviceset="PUSH-SWITCH" device="" value="PUSH-SWITCH"/>
-<part name="BTN_USR" library="SobieskiSat2" deviceset="PUSH-SWITCH" device="" value="PUSH-SWITCH"/>
+<part name="BTN_RST" library="SobieskiSat2" deviceset="PUSH-SWITCH" device="" override_package3d_urn="urn:adsk.eagle:package:21280724/2" override_package_urn="urn:adsk.eagle:footprint:21280725/1" value="PUSH-SWITCH"/>
+<part name="BTN_USR" library="SobieskiSat2" deviceset="PUSH-SWITCH" device="" override_package3d_urn="urn:adsk.eagle:package:21280593/2" override_package_urn="urn:adsk.eagle:footprint:21280594/1" value="PUSH-SWITCH"/>
 <part name="C16" library="Unified" deviceset="CAPACITOR" device="0603" package3d_urn="urn:adsk.eagle:package:23616/2" value="4.7u"/>
 <part name="U$8" library="SobieskiSat2" deviceset="BMP280" device="" package3d_urn="urn:adsk.eagle:package:16206910/2"/>
@@
 <part name="U$22" library="SobieskiSat2" deviceset="LOGO" device="RICK"/>
 <part name="GND47" library="supply1" library_urn="urn:adsk.eagle:library:371" deviceset="GND" device=""/>
-<part name="U$3" library="SobieskiSat2" deviceset="L86" device=""/>
+<part name="U$3" library="SobieskiSat2" deviceset="L86" device="" override_package3d_urn="urn:adsk.eagle:package:21280947/2" override_package_urn="urn:adsk.eagle:footprint:21280948/1"/>
 <part name="GND14" library="supply1" library_urn="urn:adsk.eagle:library:371" deviceset="GND" device=""/>
 <part name="R24" library="Unified" deviceset="RESISTOR" device="0603" package3d_urn="urn:adsk.eagle:package:23555/3" value="0R"/>
@@
 <part name="U$15" library="SobieskiSat2" deviceset="RESISTORARRAY" device="" package3d_urn="urn:adsk.eagle:package:16308440/2"/>
 <part name="U$4" library="SobieskiSat2" deviceset="RESISTORARRAY" device="" package3d_urn="urn:adsk.eagle:package:16308440/2"/>
-<part name="BTN_USR1" library="SobieskiSat2" deviceset="PUSH-SWITCH" device="" value="PUSH-SWITCH"/>
+<part name="BTN_USR1" library="SobieskiSat2" deviceset="PUSH-SWITCH" device="" override_package3d_urn="urn:adsk.eagle:package:21280924/2" override_package_urn="urn:adsk.eagle:footprint:21280925/1" value="PUSH-SWITCH"/>
 <part name="U$19" library="Unified" deviceset="CONNECTOR_F_X3" device="_JST_SMD"/>
-<part name="U$20" library="Unified" deviceset="CONNECTOR_F_X3" device="_JST_SMD"/>
+<part name="U$20" library="Unified" deviceset="CONNECTOR_F_X3" device="_JST_SMD" override_package3d_urn="urn:adsk.eagle:package:21280605/2" override_package_urn="urn:adsk.eagle:footprint:21280606/1"/>
 <part name="X1" library="SobieskiSat2" deviceset="FH12-24S-0.5S" device="H" package3d_urn="urn:adsk.eagle:package:7312/1"/>
 <part name="U$26" library="SobieskiSat2" deviceset="RESISTORARRAY" device="" package3d_urn="urn:adsk.eagle:package:16308440/2"/>
@@
 <part name="C19" library="Unified" deviceset="CAPACITOR" device="1206" package3d_urn="urn:adsk.eagle:package:23618/2" value="10u"/>
 <part name="C25" library="Unified" deviceset="CAPACITOR" device="1206" package3d_urn="urn:adsk.eagle:package:23618/2" value="10u"/>
-<part name="U$17" library="SobieskiSat2" deviceset="MOTOR_DUO" device=""/>
+<part name="U$17" library="SobieskiSat2" deviceset="MOTOR_DUO" device="" override_package3d_urn="urn:adsk.eagle:package:21280618/2" override_package_urn="urn:adsk.eagle:footprint:21280619/1"/>
 <part name="GND53" library="supply1" library_urn="urn:adsk.eagle:library:371" deviceset="GND" device=""/>
-<part name="U$13" library="SobieskiSat2" deviceset="MOTOR_DUO" device=""/>
+<part name="U$13" library="SobieskiSat2" deviceset="MOTOR_DUO" device="" override_package3d_urn="urn:adsk.eagle:package:21280931/2" override_package_urn="urn:adsk.eagle:footprint:21280932/1"/>
 <part name="GND54" library="supply1" library_urn="urn:adsk.eagle:library:371" deviceset="GND" device=""/>
 <part name="GND55" library="supply1" library_urn="urn:adsk.eagle:library:371" deviceset="GND" device=""/>
@@
 <part name="C27" library="Unified" deviceset="CAPACITOR" device="0603" package3d_urn="urn:adsk.eagle:package:23616/2" value="50p"/>
 <part name="C28" library="rcl" library_urn="urn:adsk.eagle:library:334" deviceset="CPOL-US" device="153CLV-0405" package3d_urn="urn:adsk.eagle:package:23397/2"/>
-<part name="U$14" library="SobieskiSat2" deviceset="BAT_JST_4(3)" device=""/>
+<part name="U$14" library="SobieskiSat2" deviceset="BAT_JST_4(3)" device="" override_package3d_urn="urn:adsk.eagle:package:21280658/2" override_package_urn="urn:adsk.eagle:footprint:21280659/1"/>
 <part name="R10" library="Unified" deviceset="RESISTOR" device="0603" package3d_urn="urn:adsk.eagle:package:23555/3" value="0R"/>
 <part name="GND36" library="supply1" library_urn="urn:adsk.eagle:library:371" deviceset="GND" device=""/>
 <part name="GND41" library="supply1" library_urn="urn:adsk.eagle:library:371" deviceset="GND" device=""/>
-<part name="GND51" library="supply1" library_urn="urn:adsk.eagle:library:371" deviceset="GND" device=""/>
 <part name="GND56" library="supply1" library_urn="urn:adsk.eagle:library:371" deviceset="GND" device=""/>
 <part name="GND57" library="supply1" library_urn="urn:adsk.eagle:library:371" deviceset="GND" device=""/>
 <part name="GND58" library="supply1" library_urn="urn:adsk.eagle:library:371" deviceset="GND" device=""/>
+<part name="GND59" library="supply1" library_urn="urn:adsk.eagle:library:371" deviceset="GND" device=""/>
 </parts>
 <sheets>
@@
 <attribute name="VALUE" x="254" y="-144.78" size="1.778" layer="96" align="center"/>
 </instance>
-<instance part="GND51" gate="1" x="245.11" y="-153.67" smashed="yes" rot="MR0">
-<attribute name="VALUE" x="245.11" y="-156.21" size="1.778" layer="96" rot="R90" align="center"/>
-</instance>
 <instance part="GND56" gate="1" x="278.13" y="-153.67" smashed="yes" rot="MR0">
 <attribute name="VALUE" x="278.13" y="-156.21" size="1.778" layer="96" rot="R90" align="center"/>
@@
 <instance part="GND58" gate="1" x="388.62" y="-137.16" smashed="yes" rot="MR90">
 <attribute name="VALUE" x="386.08" y="-137.16" size="1.778" layer="96" align="center"/>
+</instance>
+<instance part="GND59" gate="1" x="255.27" y="-101.6" smashed="yes" rot="MR0">
+<attribute name="VALUE" x="255.27" y="-104.14" size="1.778" layer="96" rot="R90" align="center"/>
 </instance>
 </instances>
@@
 </segment>
 <segment>
-<pinref part="GND51" gate="1" pin="GND"/>
-<pinref part="U$19" gate="G$1" pin="S$1"/>
-</segment>
-<segment>
 <pinref part="GND56" gate="1" pin="GND"/>
 <pinref part="U$20" gate="G$1" pin="S$1"/>
@@
 <pinref part="GND58" gate="1" pin="GND"/>
 <pinref part="X1" gate="G$2" pin="S$1"/>
+</segment>
+<segment>
+<pinref part="GND59" gate="1" pin="GND"/>
+<pinref part="C28" gate="G$1" pin="-"/>
 </segment>
 </net>
@@
 <wire x1="-76.2" y1="86.36" x2="-73.66" y2="86.36" width="0.1524" layer="91"/>
 <label x="-73.66" y="86.36" size="1.778" layer="95" xref="yes"/>
+</segment>
+<segment>
+<pinref part="C28" gate="G$1" pin="+"/>
+<wire x1="255.27" y1="-91.44" x2="255.27" y2="-88.9" width="0.1524" layer="91"/>
+<wire x1="255.27" y1="-88.9" x2="254" y2="-88.9" width="0.1524" layer="91"/>
+<label x="254" y="-88.9" size="1.778" layer="95" rot="R180" xref="yes"/>
+</segment>
+<segment>
+<pinref part="U$19" gate="G$1" pin="S$1"/>
+<wire x1="245.11" y1="-151.13" x2="245.11" y2="-153.67" width="0.1524" layer="91"/>
+<label x="245.11" y="-153.67" size="1.778" layer="95" rot="R270" xref="yes"/>
 </segment>
 </net>
@@
 packages will not be understood (or retained) with this version.
 </note>
+<note version="9.4" severity="warning">
+Since Version 9.4, EAGLE supports the overriding of 3D packages
+in schematics and board files. Those overridden 3d packages
+will not be understood (or retained) with this version.
+</note>
 <note version="8.4" severity="warning">

Commit message: Extension board
Parts:
- added U$18: LOGOSQSM, SobieskiSat2:LOGOSQSM
Connections:
- net GND: now also X1-18.1, X1-24.1; no longer U$25.P$9, X1-17.1, X1-23.1
- net PWM_3: no longer U$25.P$7
- net PWM_4: no longer U$25.P$8
- net VCC: now also X1-17.1, X1-23.1; no longer X1-18.1, X1-24.1

Commit message: Before ordering
Parts:
- removed C10: 10n, Unified:CAPACITOR0603
- removed C2: 10u, Unified:CAPACITOR0603
- removed C81: 100n, Unified:CAPACITOR0603
- removed R10: 0R, Unified:RESISTOR0603
- removed U$23: LOGOSQSM, SobieskiSat2:LOGOSQSM
- BTN_DFU: value SLIDE-SWITCH -> SLIDE-SWITCH2; device SobieskiSat2:SLIDE-SWITCH -> SobieskiSat2:SLIDE-SWITCH2
- U$22: value LOGORICK -> PADSMALL; device SobieskiSat2:LOGORICK -> Unified:PADSMALL
Connections:
- removed net N$25: BTN_DFU.P$1, R10.1
- net BAT: no longer C10.1
- net GND: no longer C10.2, C2.2, C81.2
- net GPS_RST: now also U$22.1; no longer R10.2
- net PWM_4: now also U$11.EN_A; no longer U$11.PH_B
- net P_EN_4: now also U$11.PH_B; no longer U$11.EN_A
- net VCC: no longer C81.1
- net VSYS: no longer C2.1
Other:
- note added: "Changes: > GPS change > LED pins change > Pads change (servo, pwm) > (no 2.4GHz radio support) > Motor driver change > Expansion connector added > USB-C changed to 2.0 > New connectors"
- note removed: "Changes: > GPS change > LED pins change > Pads change (servo, pwm) > (no 2.4GHz radio support)"
- moved on the sheet: BTN_USR, BTN_USR1, C17, C18, C19, C25, C26, C27, C28, C5, C70, C71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

Commit message: Ordered
Parts:
- removed U$22: PADSMALL, Unified:PADSMALL
Connections:
- removed net GPS_RST: U$22.1, U$3.RST
- removed net N$16: BTN_USR1.P$1, U$16G$3.2
- new net N$25: BTN_USR1.P$1, U$16G$2.2
- net DFU: now also U$16G$3.2; no longer U$16G$2.2
- net GND: now also BTN_DFU.S$1, U$16G$3.1; no longer BTN_DFU.P$2
- net NRST: now also U$3.RST
- net VCC: now also BTN_DFU.P$2; no longer U$16G$3.1
Other:
- moved on the sheet: U$16G$2, U$16G$3
Changed lines of the file:
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@@
 <part name="C11" library="Unified" deviceset="CAPACITOR" device="0603" package3d_urn="urn:adsk.eagle:package:23616/2" value="100n"/>
 <part name="P+5" library="supply1" library_urn="urn:adsk.eagle:library:371" deviceset="VCC" device=""/>
-<part name="P+6" library="supply1" library_urn="urn:adsk.eagle:library:371" deviceset="VCC" device=""/>
 <part name="GND8" library="supply1" library_urn="urn:adsk.eagle:library:371" deviceset="GND" device=""/>
 <part name="C12" library="Unified" deviceset="CAPACITOR" device="0603" package3d_urn="urn:adsk.eagle:package:23616/2" value="15p"/>
@@
 <part name="C18" library="Unified" deviceset="CAPACITOR" device="0603" package3d_urn="urn:adsk.eagle:package:23616/2" value="100n"/>
 <part name="R8" library="Unified" deviceset="RESISTOR" device="0603" package3d_urn="urn:adsk.eagle:package:23555/3" value="1k"/>
-<part name="GND9" library="supply1" library_urn="urn:adsk.eagle:library:371" deviceset="GND" device=""/>
 <part name="U$25" library="SobieskiSat2" deviceset="GPIO_DEBUG" device=""/>
 <part name="GND52" library="supply1" library_urn="urn:adsk.eagle:library:371" deviceset="GND" device=""/>
@@
 <part name="P+25" library="supply1" library_urn="urn:adsk.eagle:library:371" deviceset="VCC" device=""/>
 <part name="U$18" library="SobieskiSat2" deviceset="LOGO" device="SQSM"/>
-<part name="U$22" library="Unified" deviceset="PAD" device="SMALL" value="PADSMALL"/>
+<part name="GND51" library="supply1" library_urn="urn:adsk.eagle:library:371" deviceset="GND" device=""/>
+<part name="P+6" library="supply1" library_urn="urn:adsk.eagle:library:371" deviceset="VCC" device=""/>
+<part name="GND9" library="supply1" library_urn="urn:adsk.eagle:library:371" deviceset="GND" device=""/>
 </parts>
 <sheets>
@@
 <attribute name="VALUE" x="-54.61" y="49.53" size="1.778" layer="96" align="center"/>
 </instance>
-<instance part="P+6" gate="VCC" x="-53.34" y="66.04" smashed="yes" rot="R90">
-<attribute name="VALUE" x="-55.88" y="66.04" size="1.778" layer="96" align="center"/>
-</instance>
 <instance part="GND8" gate="1" x="-52.07" y="59.69" smashed="yes" rot="R270">
 <attribute name="VALUE" x="-54.61" y="59.69" size="1.778" layer="96" align="center"/>
@@
 <attribute name="NAME" x="72.39" y="87.122" size="1.778" layer="95" rot="MR0"/>
 </instance>
-<instance part="U$16" gate="G$2" x="-38.1" y="66.04" smashed="yes">
-<attribute name="NAME" x="-43.18" y="62.992" size="1.778" layer="95"/>
-</instance>
-<instance part="U$16" gate="G$3" x="68.58" y="3.81" smashed="yes" rot="MR0">
-<attribute name="NAME" x="73.66" y="0.762" size="1.778" layer="95" rot="MR0"/>
+<instance part="U$16" gate="G$2" x="69.85" y="3.81" smashed="yes" rot="MR0">
+<attribute name="NAME" x="74.93" y="0.762" size="1.778" layer="95" rot="MR0"/>
+</instance>
+<instance part="U$16" gate="G$3" x="-34.29" y="66.04" smashed="yes">
+<attribute name="NAME" x="-39.37" y="62.992" size="1.778" layer="95"/>
 </instance>
 <instance part="U$16" gate="G$4" x="67.31" y="1.27" smashed="yes">
@@
 <attribute name="NAME" x="-175.26" y="60.96" size="1.778" layer="95" rot="R90"/>
 <attribute name="VALUE" x="-175.26" y="72.39" size="1.778" layer="96" rot="R90"/>
-</instance>
-<instance part="GND9" gate="1" x="-53.34" y="81.28" smashed="yes">
-<attribute name="VALUE" x="-53.34" y="80.01" size="1.778" layer="96" rot="R180" align="center"/>
 </instance>
 <instance part="U$25" gate="G$1" x="-44.45" y="19.05" smashed="yes"/>
@@
 </instance>
 <instance part="U$18" gate="G$1" x="87.63" y="-13.97" smashed="yes"/>
-<instance part="U$22" gate="G$1" x="-59.69" y="73.66" smashed="yes" rot="R180"/>
+<instance part="GND51" gate="1" x="-48.26" y="66.04" smashed="yes" rot="R270">
+<attribute name="VALUE" x="-49.53" y="66.04" size="1.778" layer="96" rot="R90" align="center"/>
+</instance>
+<instance part="P+6" gate="VCC" x="-53.34" y="81.28" smashed="yes" rot="R180">
+<attribute name="VALUE" x="-53.34" y="78.74" size="1.778" layer="96" rot="R90" align="center"/>
+</instance>
+<instance part="GND9" gate="1" x="-59.69" y="86.36" smashed="yes" rot="R270">
+<attribute name="VALUE" x="-60.96" y="86.36" size="1.778" layer="96" rot="R90" align="center"/>
+</instance>
 </instances>
 <busses>
@@
 </segment>
 <segment>
-<pinref part="P+6" gate="VCC" pin="VCC"/>
-<wire x1="-43.18" y1="66.04" x2="-50.8" y2="66.04" width="0.1524" layer="91"/>
-<pinref part="U$16" gate="G$2" pin="1"/>
-</segment>
-<segment>
 <pinref part="U$8" gate="G$1" pin="VDDIO"/>
 <wire x1="-21.59" y1="-50.8" x2="-19.05" y2="-50.8" width="0.1524" layer="91"/>
@@
 </segment>
 <segment>
-<pinref part="U$16" gate="G$3" pin="1"/>
 <pinref part="P+15" gate="VCC" pin="VCC"/>
-<wire x1="73.66" y1="3.81" x2="74.93" y2="3.81" width="0.1524" layer="91"/>
 <wire x1="74.93" y1="3.81" x2="74.93" y2="2.54" width="0.1524" layer="91"/>
 <wire x1="74.93" y1="2.54" x2="74.93" y2="1.27" width="0.1524" layer="91"/>
@@
 <pinref part="U$16" gate="G$4" pin="2"/>
 <wire x1="72.39" y1="1.27" x2="74.93" y2="1.27" width="0.1524" layer="91"/>
+<pinref part="U$16" gate="G$2" pin="1"/>
 </segment>
 <segment>
@@
 <wire x1="181.61" y1="-58.42" x2="185.42" y2="-58.42" width="0.1524" layer="91"/>
 <pinref part="X1" gate="-23" pin="1"/>
+</segment>
+<segment>
+<pinref part="P+6" gate="VCC" pin="VCC"/>
+<pinref part="BTN_DFU" gate="G$1" pin="P$2"/>
 </segment>
 </net>
@@
 </segment>
 <segment>
-<pinref part="GND9" gate="1" pin="GND"/>
-<pinref part="BTN_DFU" gate="G$1" pin="P$2"/>
-</segment>
-<segment>
 <wire x1="-48.26" y1="25.4" x2="-52.07" y2="25.4" width="0.1524" layer="91"/>
 <pinref part="GND52" gate="1" pin="GND"/>
@@
 <wire x1="181.61" y1="-60.96" x2="185.42" y2="-60.96" width="0.1524" layer="91"/>
 <pinref part="X1" gate="-24" pin="1"/>
+</segment>
+<segment>
+<pinref part="GND51" gate="1" pin="GND"/>
+<pinref part="U$16" gate="G$3" pin="1"/>
+<wire x1="-39.37" y1="66.04" x2="-45.72" y2="66.04" width="0.1524" layer="91"/>
+</segment>
+<segment>
+<pinref part="GND9" gate="1" pin="GND"/>
+<pinref part="BTN_DFU" gate="G$1" pin="S$1"/>
 </segment>
 </net>
@@
 <label x="182.88" y="-33.02" size="0.762" layer="95" rot="R180" xref="yes"/>
 </segment>
+<segment>
+<pinref part="U$3" gate="G$1" pin="RST"/>
+<wire x1="255.27" y1="-49.53" x2="245.11" y2="-49.53" width="0.1524" layer="91"/>
+<label x="245.11" y="-49.53" size="1.778" layer="95"/>
+</segment>
 </net>
 <net name="DFU" class="0">
 <segment>
 <wire x1="-29.21" y1="66.04" x2="-29.21" y2="72.39" width="0.1524" layer="91"/>
-<wire x1="-33.02" y1="66.04" x2="-29.21" y2="66.04" width="0.1524" layer="91"/>
 <pinref part="U$1" gate="STM32F405RGT6_UTL" pin="BOOT0"/>
 <wire x1="7.62" y1="72.39" x2="-29.21" y2="72.39" width="0.1524" layer="91"/>
 <junction x="-29.21" y="72.39"/>
 <label x="-2.54" y="72.39" size="1.778" layer="95"/>
-<pinref part="U$16" gate="G$2" pin="2"/>
 <pinref part="BTN_DFU" gate="G$1" pin="P$3"/>
 <wire x1="-50.8" y1="83.82" x2="-50.8" y2="72.39" width="0.1524" layer="91"/>
 <wire x1="-50.8" y1="72.39" x2="-29.21" y2="72.39" width="0.1524" layer="91"/>
+<pinref part="U$16" gate="G$3" pin="2"/>
 </segment>
 <segment>
@@
 </segment>
 </net>
-<net name="N$16" class="0">
-<segment>
-<pinref part="BTN_USR1" gate="G$1" pin="P$1"/>
-<pinref part="U$16" gate="G$3" pin="2"/>
-<wire x1="62.23" y1="3.81" x2="63.5" y2="3.81" width="0.1524" layer="91"/>
-</segment>
-</net>
 <net name="N$29" class="0">
 <segment>
@@
 <wire x1="137.16" y1="-60.96" x2="135.89" y2="-60.96" width="0.1524" layer="91"/>
 <label x="135.89" y="-60.96" size="0.762" layer="95" rot="R180" xref="yes"/>
-</segment>
-</net>
-<net name="GPS_RST" class="0">
-<segment>
-<pinref part="U$3" gate="G$1" pin="RST"/>
-<wire x1="255.27" y1="-49.53" x2="245.11" y2="-49.53" width="0.1524" layer="91"/>
-<label x="245.11" y="-49.53" size="1.778" layer="95"/>
-</segment>
-<segment>
-<label x="-55.88" y="66.04" size="1.778" layer="95" rot="R270" xref="yes"/>
-<wire x1="-55.88" y1="73.66" x2="-55.88" y2="66.04" width="0.1524" layer="91"/>
-<pinref part="U$22" gate="G$1" pin="1"/>
 </segment>
 </net>
@@
 </segment>
 </net>
+<net name="N$25" class="0">
+<segment>
+<pinref part="BTN_USR1" gate="G$1" pin="P$1"/>
+<wire x1="62.23" y1="3.81" x2="64.77" y2="3.81" width="0.1524" layer="91"/>
+<pinref part="U$16" gate="G$2" pin="2"/>
+</segment>
+</net>
